Commit message: 接入底盘imu接口

File: src/dashgo_driver_ros2/urdf/dashgo_visual.urdf (robot description, URDF)
Before this commit: robot dashgo, 6 links, 5 joints
Links:
- added link imu_link; visual box size=0.03 0.03 0.01
Joints:
- added joint imu_joint: type fixed, parent base_link, child imu_link, origin xyz=0.0 0.0 0.30 rpy=0 0 0
